File: Lighting_Daughter_Back.kicad_sch (KiCad schematic)
At the start: 0 parts

Commit message: driver controls + lighting architecture
Changed lines of the file:
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@@
 	(generator_version "9.0")
 	(paper "A4")
-	(hierarchical_label "+Shunt"
-		(shape input)
-		(at 157.48 92.71 0)
+	(hierarchical_label "RRRT_BRK_Turn"
+		(shape output)
+		(at 127 96.52 0)
 		(effects
 			(font
@@
 		)
 	)
-	(hierarchical_label "-Shunt"
-		(shape input)
-		(at 157.48 97.79 0)
+	(hierarchical_label "RRLT_BRK_Turn"
+		(shape output)
+		(at 127 92.71 0)
 		(effects
 			(font
