File: Pedal_Board.kicad_sch (KiCad schematic)
At the start: 0 parts

Commit message: update pedals
Changed lines of the file:
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@@
 	(generator_version "9.0")
 	(paper "A4")
-	(hierarchical_label "+3.3V_Accel"
-		(shape output)
-		(at 108.585 78.105 0)
+	(hierarchical_label "Brake_Fluid"
+		(shape input)
+		(at 109.22 95.25 0)
 		(effects
 			(font
@@
 		)
 	)
-	(hierarchical_label "+3.3V_Brake"
-		(shape output)
-		(at 108.585 99.06 0)
+	(hierarchical_label "Accel_Pot"
+		(shape input)
+		(at 109.22 85.09 0)
 		(effects
 			(font
@@
 		)
 	)
-	(hierarchical_label "GND_Accel"
-		(shape output)
-		(at 108.585 92.075 0)
+	(hierarchical_label "Brake_Pot"
+		(shape input)
+		(at 109.22 90.17 0)
 		(effects
 			(font
-				(size 1.27 1.27)
-				(bold yes)
-			)
-			(justify left)
-		)
-	)
-	(hierarchical_label "GND_Brake"
-		(shape output)
-		(at 108.585 113.03 0)
-		(effects
-			(font
-				(size 1.27 1.27)
-				(bold yes)
-			)
-			(justify left)
-		)
-	)
-	(hierarchical_label "Sens_Accel"
-		(shape input)
-		(at 108.585 85.09 0)
-		(effects
-			(font
-				(size 1.27 1.27)
-				(bold yes)
-			)
-			(justify left)
-		)
-	)
-	(hierarchical_label "Sens_Brake"
-		(shape input)
-		(at 108.585 106.045 0)
-		(effects
-			(font
