File: Backup_Camera.kicad_sch (KiCad schematic)
At the start: 0 parts

Commit message: driver controls + lighting architecture
Changed lines of the file:
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@@
 	(generator_version "9.0")
 	(paper "A4")
-	(hierarchical_label "TemperatureTaps"
-		(shape input)
-		(at 157.48 92.71 0)
+	(hierarchical_label "USB"
+		(shape output)
+		(at 149.86 102.87 0)
 		(effects
 			(font
