File: Lighting_Daughter_Canopy.kicad_sch (KiCad schematic)
At the start: 0 parts

Commit message: driver controls + lighting architecture
Changed lines of the file:
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@@
 	(generator_version "9.0")
 	(paper "A4")
-	(hierarchical_label "TemperatureTaps"
-		(shape input)
-		(at 157.48 92.71 0)
+	(hierarchical_label "BRK_Canopy"
+		(shape output)
+		(at 127 92.71 0)
 		(effects
 			(font

Commit message: hehe
Changed lines of the file:
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@@
 	(generator_version "9.0")
 	(paper "A4")
+	(hierarchical_label "BPS_Strobe"
+		(shape output)
+		(at 127 97.79 0)
+		(effects
+			(font
+				(size 1.27 1.27)
+			)
+			(justify left)
+		)
+	)
 	(hierarchical_label "BRK_Canopy"
 		(shape output)
