File: ElectricalSystem.kicad_sch (KiCad schematic)
At the start: 6 parts, among them M1 Motor_BLDC, SW3 Supp_Enable

Commit message: hehe
Other:
- sheet Lighting_Daughter_Canopy ports: added BPS_Strobe; removed none
- note added: "add array contactor and 2 fan conns"
- note added: "combine volttemp (1-8)"
Changed lines of the file:
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@@
 		)
 	)
+	(text "add array contactor and 2 fan conns"
+		(exclude_from_sim no)
+		(at 183.388 117.348 0)
+		(effects
+			(font
+				(size 1.27 1.27)
+				(thickness 0.254)
+				(bold yes)
+				(color 255 0 0 1)
+			)
+		)
+	)
 	(text "Lighting"
 		(exclude_from_sim no)
@@
 		)
 	)
+	(text "combine volttemp (1-8)"
+		(exclude_from_sim no)
+		(at 237.236 58.928 0)
+		(effects
+			(font
+				(size 1.27 1.27)
+				(thickness 0.254)
+				(bold yes)
+				(color 255 0 0 1)
+			)
+		)
+	)
 	(text "CarCAN"
 		(exclude_from_sim no)
@@
 		)
 		(pin "BRK_Canopy" output
-			(at 400.685 93.345 180)
+			(at 400.685 92.71 180)
 			(effects
 				(font
@@
 			)
 		)
+		(pin "BPS_Strobe" output
+			(at 431.8 92.71 0)
+			(effects
+				(font
+					(size 1.27 1.27)
+				)
+				(justify right)
+			)
+		)

Commit message: stuff
Parts:
- M1: value Motor_BLDC -> Mitsuba M2096-III Motor
Other:
- note added: "HV+ Contactor"
- note added: "HV- Contactor"
- note added: "PCAN_Telemetry"
- note added: "The main CAN bus is CarCAN, which is utilized for system-wide communication (EX....). There are four peripheral CAN (PCAN) buses: BPS (Battery Protection System), Controls, Telemetry, and Motor (between VCU and motor controller)."
- note added: "add leader (+ wireless stuff), dynamics + linpot (4x), environment (6x??), TPMS transceiver (4x), broker?"
- note removed: "The main CAN bus is CarCAN, which is utilized for system-wide communication (EX....). There are three? peripheral CAN (PCAN) buses: BPS (Battery Protection System), CaT (Driver Controls & Telemetry), and Motor (between VCU and motor controller)."
- note removed: "add dynamics + linpot, environment, TPMS transceiver, broker?"
- note removed: "not sure if any of this needs isolation - check again!"
- moved on the sheet: M1

Commit message: bps leader
Connections:
- net SupplementalBattery/+12V_Supp: now also SW3.1 (A)
Other:
- sheet BPS_Daughter ports: added +Sens_ARR, -Sens_ARR, Drive_ARR, Fan1, Fan2, GND_ARR; removed none
- note added: "Array Contactor"
- note added: "Radiator Fans"
- note added: "Ventilation Fans"
- note added: "add shunt?"
- note added: "this strobe is over CAN now.."
- note removed: "add array contactor and 2 fan conns"

Commit message: whats a vcu
Other:
- sheet VehicleControlUnit ports: added +Sens_APCHG, +Sens_MPCHG, +Sens_MTR, -Sens_APCHG, -Sens_MPCHG, -Sens_MTR, Drive_APCHG, Drive_MPCHG, Drive_MTR, GND_APCHG, GND_MPCHG, GND_MTR; removed none
- note added: "Array Precharge Contactor"
- note added: "Motor Contactor"
- note added: "Motor Precharge Contactor"
- note removed: "add motor, motorpre, arraypre contactor drive/sense"
- moved on the sheet: M1

Commit message: more bps
Other:
- sheet Voltage_Daughter renamed VoltTemp_Daughter (8x)
- removed sheet PeripheralSOM2
- removed sheet Temp_Daughter
- added sheet LeaderSOM4 (LeaderSOM.kicad_sch)
- added sheet Telemetry Daughter (Wireless Transceiver) (Telemetry_Daughter.kicad_sch)
- sheet VoltTemp_Daughter (8x): file Voltage_Daughter.kicad_sch -> VoltTemp_Daughter.kicad_sch
- sheet VoltTemp_Daughter (8x) ports: added TemperatureTaps; removed none
- note added: "8 VoltTemp boards - one per battery segment (?? modules, ?? cells)."
- note added: "Wireless"
- note added: "define what we mean by HV, HC...."
- note removed: "combine volttemp (1-8)"

Commit message: contactors?
Parts:
- added K1: HV+ Contactor, symbol Relay:Relay_SPST-NO
- added K2: HV- Contactor, symbol Relay:Relay_SPST-NO
- added K3: Array Contactor, symbol Relay:Relay_SPST-NO
- added K4: Array Precharge Contactor, symbol Relay:Relay_SPST-NO
- added K5: Motor Precharge Contactor, symbol Relay:Relay_SPST-NO
- added K6: Motor Contactor, symbol Relay:Relay_SPST-NO
Connections:
- net +Sens_APCHG: now also K4.S2
- net +Sens_ARR: now also K3.S2
- net +Sens_HV+: now also K1.S2
- net +Sens_HV-: now also K2.S2
- net +Sens_MPCHG: now also K5.S2
- net +Sens_MTR: now also K6.S2
- net -Sens_APCHG: now also K4.S1
- net -Sens_ARR: now also K3.S1
- net -Sens_HV+: now also K1.S1
- net -Sens_HV-: now also K2.S1
- net -Sens_MPCHG: now also K5.S1
- net -Sens_MTR: now also K6.S1
- net Drive_APCHG: now also K4.D2
- net Drive_ARR: now also K3.D2
- net Drive_HV+: now also K1.D2
- net Drive_HV-: now also K2.D2
- net Drive_MPCHG: now also K5.D2
- net Drive_MTR: now also K6.D2
- net GND_APCHG: now also K4.D1
- net GND_ARR: now also K3.D1
- net GND_HV+: now also K1.D1
- net GND_HV-: now also K2.D1
- net GND_MPCHG: now also K5.D1
- net GND_MTR: now also K6.D1
Other:
- sheet MotorController renamed Prohelion WaveSculptor 22 Motor Controller
- note added: "- Controls Daughter Board - Steering board - Battery boards (internal HV?) - Telemetry sensors/leader - Array (MPPTs, Blackbody sensors) - Explain purpose of each CAN - Diagram CAN loop topology"
- note added: "Each MPPT internally fused to 8A"
- note added: "add contactors, internal battery architecture, bus bar connections, e-stops"
- note added: "add fuse - bus bar?"
- note added: "bus bar?"
- note added: "do we need more inline fuses?"
- note added: "motor fuse?"
- note removed: "- Controls Daughter Board - Steering board - Fans - Battery boards (internal HV?) - Telemetry sensors/leader - Array (MPPTs, Blackbody sensors) - VCU + MotorCAN? - Explain purpose of each CAN - Diagram CAN loop topology"
- note removed: "add contactors, internal battery architecture, bus bar connections"

Commit message: new precharge architecture
Other:
- sheet PrimaryBatteryPack1 renamed MainBatteryPack
- removed sheet BPS_Scrutineering1
- added sheet ActivePrechargeBoard_Array (ActivePrechargeBoard.kicad_sch)
- added sheet ActivePrechargeBoard_Motor (ActivePrechargeBoard.kicad_sch)
- sheet BPS_Daughter ports: added +Sens_APCHG, -Sens_APCHG, ArrayPreReady, ArrayPreSPI, Drive_APCHG, GND_APCHG; removed none
- sheet MainBatteryPack ports: added Pack_HV+, Pack_HV-; removed HV+, HV-
- sheet VehicleControlUnit ports: added none; removed +Sens_APCHG, -Sens_APCHG, Drive_APCHG, GND_APCHG
- note added: "Custom Bus Bar (cross-section?)"
- note added: "Main Battery"
- note added: "add bus bar connections, e-stops"
- note added: "change to separate precharge boards for BPS/VCU"
- note added: "this strobe is over CAN now?"
- note removed: "Determine scrut boards + voltage taps + thermistor breakouts depending on Powertrain"
- note removed: "Main Battery Pack"
- note removed: "add contactors, internal battery architecture, bus bar connections, e-stops"
- note removed: "this strobe is over CAN now.."

Commit message: some contactor stuff
Parts:
- added F1: 60A?, symbol Device:Fuse
- added R1: ???, symbol Device:R_Shunt
- added R2: ???, symbol Device:R
- K3: value Array Contactor -> Array Main Contactor
Connections:
- net +Shunt: now also R1.2
- net -Shunt: now also R1.3
- net ArrayPreRes+: now also K3.L2, K4.L1, R2.1
- net Pack_HV+: now also F1.1
- net Pack_HV-: now also R1.4
- net at K2.L2: now also R1.1
- net ArrayPreRes-: now reaches K1.L1
- net ArrayPreRes-: now also K4.L2, R2.2
- net at K1.L2: now also F1.2
Other:
- note added: "how does this connect to amperes?"
- note added: "rating?"
- note added: "value?"
