File: ElectricalSystem.kicad_sch (KiCad schematic)
At the start: 18 parts, among them K1 HV+ Contactor, K2 HV- Contactor, K3 Array Main Contactor, K4 Array Precharge Contactor, K5 Motor Precharge Contactor, K6 Motor Main Contactor, M1 Mitsuba M2096-III Motor, SW3 Supp_Enable

Commit message: start fixing stuff
Parts:
- removed SC1: Rear_SubArray, symbol Device:Solar_Cells
- removed SC2: FrontRight_SubArray, symbol Device:Solar_Cells
- added SC4: FrontRight_SubArray, symbol Device:Solar_Cells
- added SC5: Rear_SubArray, symbol Device:Solar_Cells
Connections:
- net MPPT_A/PV+: now also SC5.1 (+)
- net MPPT_A/PV-: now also SC5.2 (-)
- net MPPT_B/PV+: now also SC4.1 (+)
- net MPPT_B/PV-: now also SC4.2 (-)
- no-connect marks 1 -> 0
Other:
- removed sheet Backup_Camera
- removed sheet Controls_Daughter (Dashboard)
- removed sheet Display_Screen
- removed sheet Driver_Display
- removed sheet Dynamics_Board (3x)
- removed sheet Environment_Board (6x)
- removed sheet LeaderSOM2
- removed sheet LeaderSOM4
- removed sheet Left_Side_Camera
- removed sheet Lighting_Daughter_Back
- removed sheet Lighting_Daughter_Canopy
- removed sheet Lighting_Daughter_Front
- removed sheet Pedal_Board
- removed sheet PeripheralSOM12
- removed sheet PeripheralSOM13
- removed sheet PeripheralSOM4
- removed sheet PeripheralSOM5
- removed sheet PeripheralSOM7
- removed sheet PeripheralSOM8
- removed sheet Right_Side_Camera
- removed sheet Steering_Board
- removed sheet TPMS_Sensor (3x)
- removed sheet Telemetry Daughter (Wireless Transceiver)
- added sheet Array (Array.kicad_sch)
- added sheet Driver Controls (DriverControls.kicad_sch)
- added sheet Telemetry (Telemetry.kicad_sch)
- sheet LeaderSOM1 ports: added none; removed +12V_CarCAN, GND_CarCAN
- sheet LeaderSOM3 ports: added none; removed +12V_CarCAN, GND_CarCAN
- sheet MPPT_A ports: added +12V, GND; removed +12V_CarCAN, GND_CarCAN
- sheet MPPT_B ports: added +12V, GND; removed +12V_CarCAN, GND_CarCAN
- sheet MPPT_C ports: added +12V, GND; removed +12V_CarCAN, GND_CarCAN
- note added: "- all github comments - Controls Daughter Board (blocked) - Array Blackbody sensors"
- note added: "8 VoltTemp boards - one per battery segment (4 modules, 36 cells)."
- note removed: "- Controls Daughter Board - Array Blackbody sensors"
- note removed: "8 VoltTemp boards - one per battery segment (?? modules, ?? cells)."
- note removed: "Array"
- note removed: "Determine how many USB/whether using USB hub on canopy"
- note removed: "Determine what dashboard LEDs and buttons will be connected"
- note removed: "Driver Controls"
- note removed: "Lighting"
- note removed: "Telemetry"
- note removed: "add blackbody A/C (temp/irradiance sensors) 1 C per MPPT, 2 A per C"
- note removed: "do we need more inline fuses?"
- note removed: "fuse b/t array and mppt?"
- note removed: "how is TPMS implemented? how transmit to leader?"
- note removed: "or CarCAN??"
- note removed: "why two regen? also how do turn signals/horn interface?"
- moved on the sheet: F1, F2, R1, R2, R3, R4
