File: MPPT.kicad_sch (KiCad schematic)
At the start: 0 parts

Commit message: start fixing stuff
Changed lines of the file:
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@@
 	(generator_version "9.0")
 	(paper "A4")
-	(hierarchical_label "GND_CarCAN"
+	(hierarchical_label "GND"
 		(shape input)
-		(at 132.08 49.53 0)
+		(at 132.08 48.895 0)
 		(effects
 			(font
@@
 		)
 	)
+	(hierarchical_label "+12V"
+		(shape input)
+		(at 132.08 44.45 0)
+		(effects
+			(font
+				(size 1.27 1.27)
+			)
+			(justify left)
+		)
+	)
 	(hierarchical_label "+CarCAN"
 		(shape input)
@@
 		(effects
 			(font
-				(size 1.27 1.27)
-			)
-			(justify left)
-		)
-	)
-	(hierarchical_label "+12V_CarCAN"
-		(shape input)
-		(at 132.08 45.72 0)
-		(effects
-			(font
